Commit message: now ur5e touches the brick fixed the colliosn tag in urdf. now, the ismaltion is bloated need to fix it

File: ur5e_description/netft_probe.urdf (robot description, URDF)
Before this commit: robot netft_probe, 3 links, 2 joints
Links:
- link netft_link: geometry collision cylinder length=0.04906 radius=0.045; visual mesh filename=package://ur5e_description/meshes/end_effector/ati_netft_ga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
- link p42v_link: geometry collision box size=0.063 0.063 0.185; visual mesh filename=package://ur5e_description/meshes/end_effector/vera_p42v_ad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
Joints:
- joint tcp_joint: origin xyz=0 0 0.233668 rpy=0 0 0 -> xyz=0 0 0.185 rpy=0 0 0
